File: Hardware/SparkFun_USB_RFID_Reader.kicad_pcb (KiCad board)
At the start: 2 copper layers, 44.5 x 31.8 mm, 53 parts, among them J1 USB_C_Receptacle, J2 Conn_01x07_2.0mm, J3 Conn_01x05_2.0mm, J4 Conn_01x04, J6 Conn_01x04, Q1 MMBT2222A, U3 CH340C

Commit message: Post design review fixes
Parts:
- removed FID2, FID3: Fiducial_0.5mm, SparkFun-Aesthetic:Fiducial_0.5mm_Mask1mm
- removed G***: LOGO, SparkFun-Aesthetic:SparkFun_Logo_NoFlame_10mm
- removed G***: LOGO, SparkFun-Aesthetic:SparkFun_Logo_15mm
- removed Ref**: Val**, SparkFun-Aesthetic:OSHW_Logo_2.5mm
- removed kibuzzard-677EEA49: G***, kibuzzard-677EEA49
- removed kibuzzard-677EEB0A: G***, kibuzzard-677EEB0A
- removed kibuzzard-677EEB11: G***, kibuzzard-677EEB11
- removed kibuzzard-677EEB4C: G***, kibuzzard-677EEB4C
- removed kibuzzard-677EEB6C: G***, kibuzzard-677EEB6C
- removed kibuzzard-677EEBF5: G***, kibuzzard-677EEBF5
- removed kibuzzard-677EEC6E: G***, kibuzzard-677EEC6E
- removed kibuzzard-677EEEED: G***, kibuzzard-677EEEED
- removed kibuzzard-677EEF34: G***, kibuzzard-677EEF34
- removed kibuzzard-677EEF6B: G***, kibuzzard-677EEF6B
- removed kibuzzard-677EEFDD: G***, kibuzzard-677EEFDD
- removed kibuzzard-677EF000: G***, kibuzzard-677EF000
- removed kibuzzard-677EF00A: G***, kibuzzard-677EF00A
- removed kibuzzard-677EF067: G***, kibuzzard-677EF067
- removed kibuzzard-677EF074: G***, kibuzzard-677EF074
- removed kibuzzard-677EF080: G***, kibuzzard-677EF080
- removed kibuzzard-67819308: G***, kibuzzard-67819308
- removed kibuzzard-67901A90: G***, kibuzzard-67901A90
- removed kibuzzard-67901A9C: G***, kibuzzard-67901A9C
- added D2: DT1042-04SO, SparkFun-Semiconductor-Standard:SOT23-6, F.Cu at (136.8, 97.2)
- added F1: 6V/0.5A/1A, SparkFun-Fuse:0805, F.Cu at (136.8, 93.3)
- added J5: Conn_01x01, SparkFun-Connector:1x01, F.Cu at (141.6, 91.4)
- added J7: Conn_01x01, SparkFun-Connector:1x01, F.Cu at (141.6, 104.5)
- added JP3: SHLD, SparkFun-Jumper:Jumper_2_NC_Trace, B.Cu at (125.1, 97.2)
- added JP5: MD1, SparkFun-Jumper:Jumper_2_NO, B.Cu at (147.3, 84.8)
- added JP7: MD2, SparkFun-Jumper:Jumper_2_NO, B.Cu at (150.2, 84.8)
- added R5: 4.7k, SparkFun-Resistor:R_0603_1608Metric, F.Cu at (153.7, 101.9)
- added R6: 4.7k, SparkFun-Resistor:R_0603_1608Metric, F.Cu at (148.0, 87.3)
- added R7: 4.7k, SparkFun-Resistor:R_0603_1608Metric, F.Cu at (153.7, 92.1)
- added R8: 4.7k, SparkFun-Resistor:R_0603_1608Metric, F.Cu at (150.2, 92.1)
- added R9: 4.7k, SparkFun-Resistor:R_0603_1608Metric, F.Cu at (150.2, 101.9)
- added kibuzzard-67A3BA96: G***, kibuzzard-67A3BA96, B.Cu at (139.4, 91.4)
- added kibuzzard-67A3BC63: G***, kibuzzard-67A3BC63, B.Cu at (139.1, 104.5)
- added kibuzzard-67A3C4EF: G***, kibuzzard-67A3C4EF, F.Cu at (148.0, 111.8)
- added kibuzzard-67A3C54B: G***, kibuzzard-67A3C54B, B.Cu at (148.0, 111.1)
- added kibuzzard-67A3C602: G***, kibuzzard-67A3C602, F.Cu at (128.0, 106.6)
- added kibuzzard-67A3C61F: G***, kibuzzard-67A3C61F, B.Cu at (128.1, 104.1)
- added kibuzzard-67A3C62C: G***, kibuzzard-67A3C62C, B.Cu at (128.0, 106.6)
- added kibuzzard-67A3C638: G***, kibuzzard-67A3C638, F.Cu at (127.6, 109.2)
- added kibuzzard-67A3C648: G***, kibuzzard-67A3C648, B.Cu at (127.6, 109.2)
- added kibuzzard-67A3C651: G***, kibuzzard-67A3C651, F.Cu at (127.5, 111.8)
- added kibuzzard-67A3C660: G***, kibuzzard-67A3C660, B.Cu at (127.6, 111.8)
- added kibuzzard-67A3C66D: G***, kibuzzard-67A3C66D, F.Cu at (128.1, 104.1)
- added kibuzzard-67A3C67B: G***, kibuzzard-67A3C67B, F.Cu at (127.5, 90.2)
- added kibuzzard-67A3C68A: G***, kibuzzard-67A3C68A, B.Cu at (127.5, 90.2)
- added kibuzzard-67A3C68E: G***, kibuzzard-67A3C68E, F.Cu at (127.2, 87.6)
- added kibuzzard-67A3C696: G***, kibuzzard-67A3C696, B.Cu at (127.0, 87.6)
- added kibuzzard-67A3C6A9: G***, kibuzzard-67A3C6A9, F.Cu at (128.7, 85.1)
- added kibuzzard-67A3C6BA: G***, kibuzzard-67A3C6BA, B.Cu at (128.7, 85.1)
- added kibuzzard-67A3C6C4: G***, kibuzzard-67A3C6C4, F.Cu at (128.9, 82.5)
- added kibuzzard-67A3C6D3: G***, kibuzzard-67A3C6D3, B.Cu at (128.9, 82.5)
- added kibuzzard-67A3C764: G***, kibuzzard-67A3C764, B.Cu at (153.0, 84.8)
- added kibuzzard-67A3C76D: G***, kibuzzard-67A3C76D, B.Cu at (164.8, 97.2)
- added kibuzzard-67A3C77D: G***, kibuzzard-67A3C77D, B.Cu at (144.6, 84.8)
- added kibuzzard-67A3C793: G***, kibuzzard-67A3C793, B.Cu at (127.0, 97.2)
- C4: footprint SparkFun-Capacitor:C_0603_1608Metric_Polar -> SparkFun-Capacitor:C_0603_1608Metric
- D1: value Blue -> Green; footprint SparkFun-LED:LED_0603_1608Metric_Blue -> SparkFun-LED:LED_0603_1608Metric_Green
- FID1: moved to F.Cu
- moved FID1 42.2 mm to (137.5, 82.5), turned to 0 degrees
- moved J2 12.0 mm to (147.1, 89.7), turned to 0 degrees
- moved C3 1.35 mm to (153.7, 98.1), turned to 180 degrees
- moved C4 1.35 mm to (153.7, 96.2), turned to 180 degrees
Connections:
- C2 pad 1: 5V -> VUSB
- C3 pad 1: 5V -> VUSB
- C4 pad 1: 5V -> VUSB
- J1 pad S: unconnected-(J1-SHIELD-PadS) -> Net-(J1-SHIELD)
- J1 pad VBUS: 5V -> Net-(F1-Pad1)
- J2 pad 1: 5V -> TAG_IN_RANGE
- J2 pad 2: unconnected-(J2-Pin_2-Pad2) -> FORMAT
- J2 pad 3: LED -> DATA1
- J2 pad 5: DATA1 -> LED
- J2 pad 6: GND -> unconnected-(J2-Pin_6-Pad6)
- J2 pad 7: TAG_IN_RANGE -> VUSB
- J3 pad 2: 5V -> ~{RST}
- J6 pad 4: 5V -> VUSB
- JP1 pad 2: 5V -> VUSB
- JP2 pad 2: 5V -> VUSB
- U3 pad 16: 5V -> VUSB
- U3 pad 2: unconnected-(U3-TXD-Pad2) -> Net-(J5-Pin_1)
Routing:
- net VUSB: track 0.00 -> 90.9 mm, vias 0 -> 5
- net 5V: track 79.8 -> 0.00 mm, vias 5 -> 0
- net ~{RST}: track 0.00 -> 15.0 mm
- net Net-(F1-Pad1): track 0.00 -> 12.8 mm, vias 0 -> 3
- net FORMAT: track 0.00 -> 9.39 mm
- net Net-(J5-Pin_1): track 0.00 -> 9.35 mm, vias 0 -> 1
- net LED: track 16.1 -> 24.6 mm
- net CARD_PRESENT: track 42.5 -> 46.8 mm, vias 0 -> 1
- net DATA0: track 36.6 -> 40.8 mm, vias 0 -> 1
- net Net-(J1-SHIELD): track 0.00 -> 3.81 mm
- net GND: track 6.76 -> 9.36 mm, vias 8 -> 11
- net Net-(D2-I/O4): track 18.9 -> 20.9 mm
- net Net-(D2-I/O2): track 19.8 -> 20.8 mm
- net ANT1: track 29.2 -> 29.9 mm
- net DATA1: track 37.1 -> 37.0 mm, vias 1 -> 0
Other:
- copper layers 2 -> 4
- board text removed: "V20"

Commit message: Remove old files.
Parts:
- removed kibuzzard-67901575: G***, kibuzzard-67901575
- removed kibuzzard-6790157C: G***, kibuzzard-6790157C
- added G***: LOGO, SparkFun-Aesthetic:SparkFun_Logo_NoFlame_9mm, F.Cu at (152.1, 83.3)
- added G***: LOGO, SparkFun-Aesthetic:SparkFun_Logo_15mm, B.Cu at (146.7, 95.4)
- added kibuzzard-67A3C992: G***, kibuzzard-67A3C992, F.Cu at (153.0, 85.7)
- added kibuzzard-67A3C99A: G***, kibuzzard-67A3C99A, B.Cu at (146.7, 99.1)
- moved J7 1.59 mm to (141.6, 102.9)
- moved kibuzzard-67A3BC63 1.59 mm to (139.1, 102.9)
Routing:
- net CARD_PRESENT: track 46.8 -> 38.4 mm
- net ~{RST}: track 15.0 -> 14.3 mm
- net GND: vias 11 -> 12
Other:
- copper layers 4 -> 2
